Commit message: Update BASE and HIP_PITCH_L frames
1. Move Body/BASE frame to IMU
2. Change direction of HIP_PITCH_L to be the same as HIP_PITCH_R
3. Recalculate all data.

File: URDF/TH01/urdf/TH01.urdf (robot description, URDF)
Before this commit: robot TH01, 13 links, 12 joints
Links:
- link ANKLE_L: mass 0.00695 -> 0.00694571
- link ANKLE_R: mass 0.00695 -> 0.00694571
- link BASE_LINK: mass 13.79636 -> 13.88794
- link FEMUR_L: mass 3.7537 -> 3.75393
- link FEMUR_R: mass 3.75362 -> 3.75384
- link HIP_ABAD_L: mass 2.81778 -> 2.818
- link HIP_ABAD_R: mass 2.78771 -> 2.78794
- link TIBIA_L: mass 1.2755 -> 1.27716
- link TIBIA_R: mass 1.2755 -> 1.27716
Joints:
- joint HIP_PITCH_R: axis 0 0 -1 -> 0 0 1

Commit message: Update a bug

File: URDF/TH01/urdf/TH01.urdf (robot description, URDF)
Before this commit: robot TH01, 13 links, 12 joints
Joints:
- joint HIP_PITCH_L: origin xyz=0.029 0 0 rpy=-1.5708 0.7854 1.5708 -> xyz=0.029 0 0 rpy=-1.5708 0.7854 -1.5708
- joint HIP_ROLL_L: origin xyz=0.141 0 0 rpy=-1.5708 0 1.5708 -> xyz=0.141 0 0 rpy=1.5708 0 -1.5708

Commit message: Bug fix

File: URDF/TH01/urdf/TH01.urdf (robot description, URDF)
Before this commit: robot TH01, 13 links, 12 joints
Joints:
- joint HIP_YAW_L: origin xyz=-0.082378 0.0625 -0.082378 rpy=0 0.7854 0 -> xyz=-0.18337794 0.0625 -0.25076794 rpy=0 0.7854 0
- joint HIP_YAW_R: origin xyz=-0.082378 -0.0625 -0.082378 rpy=0 0.7854 0 -> xyz=-0.18338 -0.0625 -0.25077 rpy=0 0.7854 0

Commit message: Bug fix

File: URDF/TH01/urdf/TH01.urdf (robot description, URDF)
Before this commit: robot TH01, 13 links, 12 joints
Joints:
- joint HIP_PITCH_L: origin xyz=0.029 0 0 rpy=-1.5708 0.7854 -1.5708 -> xyz=-0.029 0 0 rpy=-1.5708 0.7854 -1.5708

Commit message: Update Body mass and inertia

File: URDF/TH01/urdf/TH01.urdf (robot description, URDF)
Before this commit: robot TH01, 13 links, 12 joints
Links:
- link BASE_LINK: mass 13.88794 -> 12.79294

Commit message: TH01-155T_031024

File: URDF/TH01/urdf/TH01.urdf (robot description, URDF)
Before this commit: robot TH01, 13 links, 12 joints
Links:
- link BASE_LINK: mass 12.79294 -> 13.94967

Commit message: URDF Update 042924

File: URDF/TH01/urdf/TH01.urdf (robot description, URDF)
Before this commit: robot TH01, 13 links, 12 joints
Links:
- link BASE_LINK: mass 13.94967 -> 13.27922
Joints:
- joint HIP_YAW_L: origin xyz=-0.18337794 0.0625 -0.25076794 rpy=0 0.7854 0 -> xyz=-0.114705815 0.0624996 -0.120801022 rpy=0 0.785398163 0
- joint HIP_YAW_R: origin xyz=-0.18338 -0.0625 -0.25077 rpy=0 0.7854 0 -> xyz=-0.114705815 -0.0625004 -0.120801022 rpy=0 0.785398163 0

Commit message: Create new record

File: URDF/TH01/urdf/TH01.urdf (robot description, URDF)
Before this commit: robot TH01, 13 links, 12 joints
Links:
- added link FOREARM_L, mass 0.084277249; collision mesh filename=package://TH01/meshes/FOREARM_L.STL; visual mesh filename=package://TH01/meshes/FOREARM_L.STL
- added link FOREARM_R, mass 0.084277249; collision mesh filename=package://TH01/meshes/FOREARM_R.STL; visual mesh filename=package://TH01/meshes/FOREARM_R.STL
- added link HEAD, mass 0.342268448; collision mesh filename=package://TH01/meshes/HEAD.STL; visual mesh filename=package://TH01/meshes/HEAD.STL
- added link LOWERSHOULDER_L, mass 0.166153725; collision mesh filename=package://TH01/meshes/LOWERSHOULDER_L.STL; visual mesh filename=package://TH01/meshes/LOWERSHOULDER_L.STL
- added link LOWERSHOULDER_R, mass 0.166153725; collision mesh filename=package://TH01/meshes/LOWERSHOULDER_R.STL; visual mesh filename=package://TH01/meshes/LOWERSHOULDER_R.STL
- added link NECK, mass 0.166812238; collision mesh filename=package://TH01/meshes/NECK.STL; visual mesh filename=package://TH01/meshes/NECK.STL
- added link UPPERARM_L, mass 0.227314115; collision mesh filename=package://TH01/meshes/UPPERARM_L.STL; visual mesh filename=package://TH01/meshes/UPPERARM_L.STL
- added link UPPERARM_R, mass 0.227025841; collision mesh filename=package://TH01/meshes/UPPERARM_R.STL; visual mesh filename=package://TH01/meshes/UPPERARM_R.STL
- added link UPPERSHOULDER_L, mass 0.191209791; collision mesh filename=package://TH01/meshes/UPPERSHOULDER_L.STL; visual mesh filename=package://TH01/meshes/UPPERSHOULDER_L.STL
- added link UPPERSHOULDER_R, mass 0.192254092; collision mesh filename=package://TH01/meshes/UPPERSHOULDER_R.STL; visual mesh filename=package://TH01/meshes/UPPERSHOULDER_R.STL
- link ANKLE_L: mass 0.00694571 -> 0.00695
- link ANKLE_R: mass 0.00694571 -> 0.00695
- link BASE_LINK: mass 12.79294 -> 17.38212369
- link FEMUR_L: mass 3.75393 -> 3.7537
- link FEMUR_R: mass 3.75384 -> 3.75362
- link HIP_ABAD_L: mass 2.818 -> 2.81778
- link HIP_ABAD_R: mass 2.78794 -> 2.78771
- link TIBIA_L: mass 1.27716 -> 1.2755
- link TIBIA_R: mass 1.27716 -> 1.2755
Joints:
- added joint ELBOW_PITCH_L: type revolute, parent UPPERARM_L, child FOREARM_L, origin xyz=0 0.0125 0.22375 rpy=0 -1.570796327 3.141592653, axis 0 0 1, limit lower=0 upper=0 effort=0 velocity=0
- added joint ELBOW_PITCH_R: type revolute, parent UPPERARM_R, child FOREARM_R, origin xyz=0 -0.0125 0.22375 rpy=0 -1.570796327 3.141592653, axis 0 0 1, limit lower=0 upper=0 effort=0 velocity=0
- added joint HEAD_PITCH: type revolute, parent NECK, child HEAD, origin xyz=0 0 0 rpy=1.570796327 0 0, axis 0 0 1, limit lower=0 upper=0 effort=0 velocity=0
- added joint HEAD_YAW: type revolute, parent BASE_LINK, child NECK, origin xyz=-0.063573305 0 0.192967296 rpy=0 0 0, axis 0 0 1, limit lower=0 upper=0 effort=0 velocity=0
- added joint SHOULDER_PITCH_L: type revolute, parent BASE_LINK, child UPPERSHOULDER_L, origin xyz=-0.101630818 0.15565 0.106737259 rpy=1.570796327 0 0, axis 0 0 1, limit lower=0 upper=0 effort=0 velocity=0
- added joint SHOULDER_PITCH_R: type revolute, parent BASE_LINK, child UPPERSHOULDER_R, origin xyz=-0.101630818 -0.15565 0.106737259 rpy=1.570796327 0 0, axis 0 0 1, limit lower=0 upper=0 effort=0 velocity=0
- added joint SHOULDER_ROLL_L: type revolute, parent UPPERSHOULDER_L, child LOWERSHOULDER_L, origin xyz=0 0 0 rpy=0 1.570796327 0, axis 0 0 1, limit lower=0 upper=0 effort=0 velocity=0
- added joint SHOULDER_ROLL_R: type revolute, parent UPPERSHOULDER_R, child LOWERSHOULDER_R, origin xyz=0 0 0 rpy=0 -1.570796327 3.141592653, axis 0 0 1, limit lower=0 upper=0 effort=0 velocity=0
- added joint SHOULDER_YAW_L: type revolute, parent LOWERSHOULDER_L, child UPPERARM_L, origin xyz=0 0 0 rpy=0 -1.570796327 3.141592653, axis 0 0 1, limit lower=0 upper=0 effort=0 velocity=0
- added joint SHOULDER_YAW_R: type revolute, parent LOWERSHOULDER_R, child UPPERARM_R, origin xyz=0 0 0 rpy=0 -1.570796327 3.141592653, axis 0 0 1, limit lower=0 upper=0 effort=0 velocity=0
- joint ANKLE_ROLL_L: origin xyz=0 0 0 rpy=-1.5708 0 0 -> xyz=0 0 0 rpy=-1.570796327 0 0
- joint ANKLE_ROLL_R: origin xyz=0 0 0 rpy=-1.5708 0 0 -> xyz=0 0 0 rpy=-1.570796327 0 0
- joint HIP_PITCH_L: origin xyz=-0.029 0 0 rpy=-1.5708 0.7854 -1.5708 -> xyz=-0.029 0 0 rpy=-1.570796327 0.785398163 -1.570796327
- joint HIP_PITCH_R: origin xyz=0.029 0 0 rpy=-1.5708 0.7854 -1.5708 -> xyz=0.029 0 0 rpy=-1.570796327 0.785398163 -1.570796327
- joint HIP_ROLL_L: origin xyz=0.141 0 0 rpy=1.5708 0 -1.5708 -> xyz=0.141 0 0 rpy=1.570796327 0 -1.570796327
- joint HIP_ROLL_R: origin xyz=0.141 0 0 rpy=1.5708 0 -1.5708 -> xyz=0.141 0 0 rpy=1.570796327 0 -1.570796327
- joint HIP_YAW_L: origin xyz=-0.18337794 0.0625 -0.25076794 rpy=0 0.7854 0 -> xyz=-0.18562794 0.0625 -0.29399794 rpy=0 0.785398163 0
- joint HIP_YAW_R: origin xyz=-0.18338 -0.0625 -0.25077 rpy=0 0.7854 0 -> xyz=-0.18562794 -0.0625 -0.29399794 rpy=0 0.785398163 0

Commit message: Bug fix

File: URDF/TH01/urdf/TH01.urdf (robot description, URDF)
Before this commit: robot TH01, 23 links, 22 joints
Links:
- link ANKLE_L: mass 0.00695 -> 0.00694571
- link ANKLE_R: mass 0.00695 -> 0.00694571
- link BASE_LINK: mass 17.38212369 -> 11.60239
- link FEMUR_L: mass 3.7537 -> 3.75393
- link FEMUR_R: mass 3.75362 -> 3.75384
- link FOOT_L: mass 0.17981 -> 0.41628
- link FOOT_R: mass 0.17981 -> 0.41628
- link FOREARM_L: mass 0.084277249 -> 0.0999
- link FOREARM_R: mass 0.084277249 -> 0.0999
- link HEAD: mass 0.342268448 -> 0.67367
- link HIP_ABAD_L: mass 2.81778 -> 2.818
- link HIP_ABAD_R: mass 2.78771 -> 2.78794
- link LOWERSHOULDER_L: mass 0.166153725 -> 0.35798
- link LOWERSHOULDER_R: mass 0.166153725 -> 0.35798
- link NECK: mass 0.166812238 -> 0.34044
- link TIBIA_L: mass 1.2755 -> 1.27716
- link TIBIA_R: mass 1.2755 -> 1.27716
- link UPPERARM_L: mass 0.227314115 -> 0.47342
- link UPPERARM_R: mass 0.227025841 -> 0.47342
- link UPPERSHOULDER_L: mass 0.191209791 -> 0.44001
- link UPPERSHOULDER_R: mass 0.192254092 -> 0.43611
Joints:
- joint ANKLE_ROLL_L: origin xyz=0 0 0 rpy=-1.570796327 0 0 -> xyz=0 0 0 rpy=-1.5708 0 0
- joint ANKLE_ROLL_R: origin xyz=0 0 0 rpy=-1.570796327 0 0 -> xyz=0 0 0 rpy=-1.5708 0 0
- joint ELBOW_PITCH_L: origin xyz=0 0.0125 0.22375 rpy=0 -1.570796327 3.141592653 -> xyz=0 0.0125 0.22375 rpy=0 -1.5708 3.141593
- joint ELBOW_PITCH_R: origin xyz=0 -0.0125 0.22375 rpy=0 -1.570796327 3.141592653 -> xyz=0 -0.0125 0.22375 rpy=0 -1.5708 3.141593
- joint HEAD_PITCH: origin xyz=0 0 0 rpy=1.570796327 0 0 -> xyz=0 0 0 rpy=1.570796 0 0
- joint HEAD_YAW: origin xyz=-0.063573305 0 0.192967296 rpy=0 0 0 -> xyz=-0.06357 0 0.192967 rpy=0 0 0
- joint HIP_PITCH_L: origin xyz=-0.029 0 0 rpy=-1.570796327 0.785398163 -1.570796327 -> xyz=-0.029 0 0 rpy=-1.5708 0.7854 -1.5708
- joint HIP_PITCH_R: origin xyz=0.029 0 0 rpy=-1.570796327 0.785398163 -1.570796327 -> xyz=0.029 0 0 rpy=-1.5708 0.7854 -1.5708
- joint HIP_ROLL_L: origin xyz=0.141 0 0 rpy=1.570796327 0 -1.570796327 -> xyz=0.141 0 0 rpy=1.5708 0 -1.5708
- joint HIP_ROLL_R: origin xyz=0.141 0 0 rpy=1.570796327 0 -1.570796327 -> xyz=0.141 0 0 rpy=1.5708 0 -1.5708
- joint HIP_YAW_L: origin xyz=-0.18562794 0.0625 -0.29399794 rpy=0 0.785398163 0 -> xyz=-0.18337794 0.0625 -0.25076794 rpy=0 0.7854 0
- joint HIP_YAW_R: origin xyz=-0.18562794 -0.0625 -0.29399794 rpy=0 0.785398163 0 -> xyz=-0.18338 -0.0625 -0.25077 rpy=0 0.7854 0
- joint SHOULDER_PITCH_L: origin xyz=-0.101630818 0.15565 0.106737259 rpy=1.570796327 0 0 -> xyz=-0.10163 0.15565 0.106737 rpy=1.570796 0 0
- joint SHOULDER_PITCH_R: origin xyz=-0.101630818 -0.15565 0.106737259 rpy=1.570796327 0 0 -> xyz=-0.10163 -0.15565 0.106737 rpy=1.570796 0 0
- joint SHOULDER_ROLL_L: origin xyz=0 0 0 rpy=0 1.570796327 0 -> xyz=0 0 0 rpy=0 1.570796 0
- joint SHOULDER_ROLL_R: origin xyz=0 0 0 rpy=0 -1.570796327 3.141592653 -> xyz=0 0 0 rpy=0 -1.5708 3.141593
- joint SHOULDER_YAW_L: origin xyz=0 0 0 rpy=0 -1.570796327 3.141592653 -> xyz=0 0 0 rpy=0 -1.5708 3.141593
- joint SHOULDER_YAW_R: origin xyz=0 0 0 rpy=0 -1.570796327 3.141592653 -> xyz=0 0 0 rpy=0 -1.5708 3.141593

Commit message: bug fix

File: URDF/TH01/urdf/TH01.urdf (robot description, URDF)
Before this commit: robot TH01, 23 links, 22 joints
Joints:
- joint HIP_YAW_L: origin xyz=-0.18337794 0.0625 -0.25076794 rpy=0 0.7854 0 -> xyz=-0.18562794 0.0625 -0.29399794 rpy=0 0.785398163 0
- joint HIP_YAW_R: origin xyz=-0.18338 -0.0625 -0.25077 rpy=0 0.7854 0 -> xyz=-0.18562794 -0.0625 -0.29399794 rpy=0 0.785398163 0

Commit message: bug fix

File: URDF/TH01/urdf/TH01.urdf (robot description, URDF)
Before this commit: robot TH01, 23 links, 22 joints
Links:
- link UPPERSHOULDER_L: mass 0.44001 -> 0.43611
