Commit message: Update mass and inertia properties.

File: TH02/urdf/archive/TH02.urdf (robot description, URDF)
Before this commit: robot TH02, 29 links, 28 joints
Links:
- link ANKLE_L: mass 0.006946 -> 0.015158989
- link ANKLE_R: mass 0.006946 -> 0.015158989
- link BASE_LINK: mass 12.72953 -> 3.774608038
- link FEMUR_L: mass 3.75393 -> 2.979880153
- link FEMUR_R: mass 3.75384 -> 2.979880153
- link FOOT_L: mass 0.41628 -> 0.371033238
- link FOOT_R: mass 0.41628 -> 0.371032918
- link FOREARM_L: mass 0.600199 -> 0.394752443
- link FOREARM_R: mass 0.600199 -> 0.394752441
- link HAND_L: mass 0.0001 -> 0.097947319
- link HAND_R: mass 0.0001 -> 0.097947319
- link HEAD: mass 0.67367 -> 0.342266182
- link HIP_ABAD_L: mass 2.818 -> 1.507235175
- link HIP_ABAD_R: mass 2.78794 -> 1.507235175
- link HIP_L: mass 0.83264 -> 0.53261465
- link HIP_R: mass 0.83264 -> 0.53261465
- link LOWERSHOULDER_L: mass 0.35798 -> 0.166153725
- link LOWERSHOULDER_R: mass 0.35798 -> 0.166153725
- link NECK: mass 0.34044 -> 0.166812257
- link TIBIA_L: mass 1.27716 -> 0.477888041
- link TIBIA_R: mass 1.27716 -> 0.477888041
- link UPPERARM_L: mass 0.947611 -> 0.570326844
- link UPPERARM_R: mass 0.948095 -> 0.570326844
- link UPPERSHOULDER_L: mass 0.43611 -> 0.191209791
- link UPPERSHOULDER_R: mass 0.43611 -> 0.192254092
- link WRIST_L: mass 0.086994 -> 0.097947319
- link WRIST_R: mass 0.086994 -> 0.097947319
- link WRIST_SHAFT_L: mass 0.066849 -> 0.009625385
- link WRIST_SHAFT_R: mass 0.066849 -> 0.009625385
