Commit message: URDF coordinate bug fix

File: TH02-A7/urdf/TH02-A7.urdf (robot description, URDF)
Before this commit: robot TH02-A7, 29 links, 28 joints
Links:
- link ANKLE_L: mass 0.015158989 -> 0.006946
- link ANKLE_R: mass 0.015158989 -> 0.006946
- link BASE_LINK: mass 3.521559545 -> 12.72953
- link ELBOW_L: mass 0.498142108 -> 
- link ELBOW_R: mass 0.498127999 -> 
- link FEMUR_L: mass 2.979880153 -> 3.75393
- link FEMUR_R: mass 2.979880153 -> 3.75384
- link FOOT_L: mass 0.371031799 -> 0.41628
- link FOOT_R: mass 0.371031474 -> 0.41628
- link FOREARM_L: mass 0.205822054 -> 
- link FOREARM_R: mass 0.205821255 -> 
- link HIP_ABAD_L: mass 1.507235175 -> 2.818
- link HIP_ABAD_R: mass 1.507235175 -> 2.78794
- link HIP_L: mass 0.53261465 -> 0.83264
- link HIP_R: mass 0.53261465 -> 0.83264
- link LOWERSHOULDER_R: mass 0.508258636 -> 0.35798
- link LOWERWRIST_L: mass 0.117272386 -> 
- link LOWERWRIST_R: mass 0.117272386 -> 
- link TIBIA_L: mass 0.477888041 -> 1.27716
- link TIBIA_R: mass 0.477888041 -> 1.27716
- link UPPERARM_L: mass 0.217903202 -> 
- link UPPERARM_R: mass 0.217903069 -> 
- link UPPERSHOULDER_L: mass 0.513230477 -> 0.35798
- link UPPERSHOULDER_R: mass 0.513230475 -> 0.43611
- link UPPERWRIST_L: mass 0.488379339 -> 
- link UPPERWRIST_R: mass 0.488379334 -> 
Joints:
- joint WRIST_PITCH_L: origin xyz=0 0 0 rpy=0 -1.570796327 0 -> xyz=0 0 0 rpy=3.141592653 -1.570796327 0
- joint WRIST_YAW_L: origin xyz=0.12675 0 0 rpy=0 1.570796327 0 -> xyz=0.12675 0 0 rpy=0 -1.570796327 3.141592653

Commit message: Update: mass and inertia, lowerwrist coordinate
Update the mass and inertia data to reflect the actual robot; Move the location of the LOWERWRIST limb to intersect its parent.

File: TH02-A7/urdf/TH02-A7.urdf (robot description, URDF)
Before this commit: robot TH02-A7, 29 links, 28 joints
Links:
- link ELBOW_L: mass  -> 0.37854
- link ELBOW_R: mass  -> 0.37853
- link FOREARM_L: mass  -> 0.47694
- link FOREARM_R: mass  -> 0.47694
- link HEAD: mass 0.342266182 -> 0.67367
- link LOWERWRIST_L: mass  -> 0.42
- link LOWERWRIST_R: mass  -> 0.42
- link NECK: mass 0.166812257 -> 0.34044
- link UPPERARM_L: mass  -> 0.50401
- link UPPERARM_R: mass  -> 0.50401
- link UPPERWRIST_L: mass  -> 0.37004
- link UPPERWRIST_R: mass  -> 0.37004
Joints:
- joint ELBOW_YAW_L: origin xyz=0.154950006 0.015 0 rpy=-3.14133862 -1.570796312 0 -> xyz=0.154950006 0.015 0 rpy=3.14133862 -1.570796312 0
- joint WRIST_YAW: origin xyz=0.12675 -5.00E-05 0 rpy=3.141592653 -1.570796327 0 -> xyz=0 0 0 rpy=3.141592653 -1.570796327 0
- joint WRIST_YAW_L: origin xyz=0.12675 0 0 rpy=0 -1.570796327 3.141592653 -> xyz=0 0 0 rpy=3.141592653 -1.570796327 0

Commit message: Fix mass & inertia data for UPPER & LOWER SHOULDER of Left

File: TH02-A7/urdf/TH02-A7.urdf (robot description, URDF)
Before this commit: robot TH02-A7, 29 links, 28 joints
Links:
- link LOWERSHOULDER_L: mass 0.508259807 -> 0.35798
- link UPPERSHOULDER_L: mass 0.35798 -> 0.43611
Joints:
- removed joint WRIST_YAW
- added joint WRIST_YAW_R: type revolute, parent UPPERWRIST_R, child LOWERWRIST_R, origin xyz=0 0 0 rpy=3.141592653 -1.570796327 0, axis 0 0 1, limit lower=0 upper=0 effort=0 velocity=0

Commit message: Update UpperArm model and data

File: TH02-A7/urdf/TH02-A7.urdf (robot description, URDF)
Before this commit: robot TH02-A7, 29 links, 28 joints
Links:
- link UPPERARM_L: mass 0.50401 -> 0.51544
- link UPPERARM_R: mass 0.50401 -> 0.51544
Joints:
- joint ELBOW_PITCH_L: origin xyz=0 0.015 0.19995 rpy=3.141592653 -1.570796327 0 -> xyz=0 0.015 0.22495 rpy=3.141592653 -1.570796327 0
- joint ELBOW_PITCH_R: origin xyz=0 -0.015 0.19995 rpy=0 -1.570796327 3.141592653 -> xyz=0 -0.015 0.22495 rpy=0 -1.570796327 3.141592653
