Commit message: Optimized robot properties.
- Optimized inertia for ANKLE and LOWER_WRIST
- Added command_effort for joints

File: TH02-A7/urdf/archive/TH02-A7.urdf (robot description, URDF)
Before this commit: robot TH02-A7, 29 links, 28 joints
Links:
- link ANKLE_L: mass 0.01 -> 0.006946
- link ANKLE_R: mass 0.01 -> 0.006946
Joints:
- joint ANKLE_PITCH_L: limit lower=-1 upper=1.5 effort=35 velocity=30 -> lower=0 upper=0 effort=0 velocity=0
- joint ANKLE_PITCH_R: limit lower=-1 upper=1.5 effort=35 velocity=30 -> lower=0 upper=0 effort=0 velocity=0
- joint ANKLE_ROLL_L: limit lower=-0.3 upper=0.3 effort=35 velocity=30 -> lower=0 upper=0 effort=0 velocity=0
- joint ANKLE_ROLL_R: limit lower=-0.3 upper=0.3 effort=35 velocity=30 -> lower=0 upper=0 effort=0 velocity=0
- joint ELBOW_PITCH_L: limit lower=-3.1416 upper=3.1416 effort=28 velocity=30 -> lower=0 upper=0 effort=0 velocity=0
- joint ELBOW_PITCH_R: limit lower=-3.1416 upper=3.1416 effort=28 velocity=30 -> lower=0 upper=0 effort=0 velocity=0
- joint ELBOW_YAW_L: limit lower=-3.1416 upper=3.1416 effort=28 velocity=30 -> lower=0 upper=0 effort=0 velocity=0
- joint ELBOW_YAW_R: limit lower=-3.1416 upper=3.1416 effort=28 velocity=30 -> lower=0 upper=0 effort=0 velocity=0
- joint HEAD_PITCH: limit lower=-1.6 upper=1.6 effort=28 velocity=30 -> lower=0 upper=0 effort=0 velocity=0
- joint HEAD_YAW: limit lower=-1.6 upper=1.6 effort=28 velocity=30 -> lower=0 upper=0 effort=0 velocity=0
- joint HIP_PITCH_L: limit lower=-1.4 upper=1.4 effort=150 velocity=30 -> lower=0 upper=0 effort=0 velocity=0
- joint HIP_PITCH_R: limit lower=-1.4 upper=1.4 effort=150 velocity=30 -> lower=0 upper=0 effort=0 velocity=0
- joint HIP_ROLL_L: limit lower=-1.4 upper=1.4 effort=150 velocity=30 -> lower=0 upper=0 effort=0 velocity=0
- joint HIP_ROLL_R: limit lower=-1.4 upper=1.4 effort=150 velocity=30 -> lower=0 upper=0 effort=0 velocity=0
- joint HIP_YAW_L: limit lower=-1.4 upper=1.4 effort=150 velocity=30 -> lower=0 upper=0 effort=0 velocity=0
- joint HIP_YAW_R: limit lower=-1.4 upper=1.4 effort=150 velocity=30 -> lower=0 upper=0 effort=0 velocity=0
- joint KNEE_PITCH_L: limit lower=-2.4 upper=-0.1 effort=150 velocity=30 -> lower=0 upper=0 effort=0 velocity=0
- joint KNEE_PITCH_R: limit lower=-2.4 upper=-0.1 effort=150 velocity=30 -> lower=0 upper=0 effort=0 velocity=0
- joint SHOULDER_PITCH_L: limit lower=-3.1416 upper=3.1416 effort=50 velocity=30 -> lower=0 upper=0 effort=0 velocity=0
- joint SHOULDER_PITCH_R: limit lower=-3.1416 upper=3.1416 effort=50 velocity=30 -> lower=0 upper=0 effort=0 velocity=0
- joint SHOULDER_ROLL_L: limit lower=-1.6 upper=1.6 effort=28 velocity=30 -> lower=0 upper=0 effort=0 velocity=0
- joint SHOULDER_ROLL_R: limit lower=-1.6 upper=1.6 effort=28 velocity=30 -> lower=0 upper=0 effort=0 velocity=0
- joint SHOULDER_YAW_L: limit lower=-3.1416 upper=3.1416 effort=28 velocity=30 -> lower=0 upper=0 effort=0 velocity=0
- joint SHOULDER_YAW_R: limit lower=-3.1416 upper=3.1416 effort=28 velocity=30 -> lower=0 upper=0 effort=0 velocity=0
- joint WRIST_PITCH_L: limit lower=-3.1416 upper=3.1416 effort=28 velocity=30 -> lower=0 upper=0 effort=0 velocity=0
- joint WRIST_PITCH_R: limit lower=-3.1416 upper=3.1416 effort=28 velocity=30 -> lower=0 upper=0 effort=0 velocity=0
- joint WRIST_YAW_L: limit lower=-3.1416 upper=3.1416 effort=28 velocity=30 -> lower=0 upper=0 effort=0 velocity=0
- joint WRIST_YAW_R: limit lower=-3.1416 upper=3.1416 effort=28 velocity=30 -> lower=0 upper=0 effort=0 velocity=0
